File: Nodo_Actuadores/Nodo_Actuadores.kicad_sch (KiCad schematic)
At the start: 0 parts

Commit message: Nodo_Sensores V1.0
Parts:
- added D1: D, symbol Device:D
- added J1: (no value), symbol Connector:Screw_Terminal_01x03
- added K1: (no value), Relay_THT:Relay_SPDT_SANYOU_SRD_Series_Form_C, symbol Relay:SANYOU_SRD_Form_C
- added Q1: NX3020NAKS, Package_TO_SOT_SMD:SOT-363_SC-70-6, symbol p6_test_perifericos:DMN63D8LDW-7
- added R1: 0, Resistor_SMD:R_0603_1608Metric, symbol Device:R
- added R2: 100, Resistor_SMD:R_0603_1608Metric, symbol Device:R
- added R3, R4: 10k, Resistor_SMD:R_0603_1608Metric, symbol Device:R
- added U1: ESP32_NODEMCU, Proyecto:MODULE_ESP32_NODEMCU, symbol ESP32_NODEMCU:ESP32_NODEMCU
- added U2: VOS615A-3T, footprints:SOIC127P700X210-4N, symbol VOS615B-3T:VOS615B-3T
Connections:
- new net: J1.1 (Pin_1), K1.1
- new net: J1.2 (Pin_2), K1.3
- new net: J1.3 (Pin_3), K1.4
- new net: R2.1, U2.2
- new net: Q1.3 (D2), R2.2
- new net: R1.2, U2.4
- new net: Q1.5 (G2), Q1.6 (D1), R4.2
- new net +3.3V: R3.1, R4.1
- new net +5V: D1.1 (K), K1.5, U2.1
- new net GND: D1.2 (A), K1.2, Q1.1 (S1), Q1.4 (S2)
- new net PWR_SW_N: U2.3
- new net PWR_SW_P: R1.1
- new net RELAY1: Q1.2 (G1), R3.2

Commit message: Nodo actuadores V1 finalizada
Parts:
- removed D1: D, symbol Device:D
- removed J1: (no value), symbol Connector:Screw_Terminal_01x03
- removed K1: (no value), Relay_THT:Relay_SPDT_SANYOU_SRD_Series_Form_C, symbol Relay:SANYOU_SRD_Form_C
- removed Q1: NX3020NAKS, Package_TO_SOT_SMD:SOT-363_SC-70-6, symbol p6_test_perifericos:DMN63D8LDW-7
- removed R1: 0, Resistor_SMD:R_0603_1608Metric, symbol Device:R
- removed R2: 100, Resistor_SMD:R_0603_1608Metric, symbol Device:R
- removed R3, R4: 10k, Resistor_SMD:R_0603_1608Metric, symbol Device:R
- removed U1: ESP32_NODEMCU, Proyecto:MODULE_ESP32_NODEMCU, symbol ESP32_NODEMCU:ESP32_NODEMCU
- removed U2: VOS615A-3T, footprints:SOIC127P700X210-4N, symbol VOS615B-3T:VOS615B-3T
- added C1 (x2): 0.1uF, Capacitor_SMD:C_0805_2012Metric, symbol Device:C
- added H1, H2, H3, H4: MountingHole, MountingHole:MountingHole_3.2mm_M3_DIN965, symbol Mechanical:MountingHole
- added J3: Conn_01x04, Connector_PinHeader_2.54mm:PinHeader_1x04_P2.54mm_Vertical, symbol Connector_Generic:Conn_01x04
- added R32 (x2): 220, Resistor_SMD:R_0805_2012Metric_Pad1.20x1.40mm_HandSolder, symbol Device:R
- added R32 (x2): 10K, Resistor_SMD:R_0805_2012Metric_Pad1.20x1.40mm_HandSolder, symbol Device:R
- added SW1: Reset, ProyectoUTN:SW_Tactile_SPST_NO_Straight_6x3,5_modificado, symbol Switch:SW_Omron_B3FS
- added SW2: Flash, ProyectoUTN:SW_Tactile_SPST_NO_Straight_6x3,5_modificado, symbol Switch:SW_Omron_B3FS
- added U3: ESP32-WROOM-32E__4MB_HIGH_TEMP_, ESP32:ESP32-WROOM-32E__4MB_HIGH_TEMP, symbol ESP32-WROOM-32E__4MB_HIGH_TEMP_:ESP32-WROOM-32E__4MB_HIGH_TEMP_
Connections:
- net GND: now also C1.1, C1.2, J3.4 (Pin_4), SW1.1, SW2.2, U3.1 (GND), U3.15 (GND), U3.38 (GND), U3.39_1 (GND), U3.39_2 (GND), U3.39_3 (GND), U3.39_4 (GND), U3.39_5 (GND), U3.39_6 (GND), U3.39_7 (GND), U3.39_8 (GND), U3.39_9 (GND)
- new net: U3.17 (NC), U3.18 (NC), U3.19 (NC), U3.20 (NC), U3.21 (NC), U3.22 (NC)
- new net: C1.2, R32.1, R32.1, U3.25 (IO0)
- new net: C1.1, R32.2, R32.2, U3.3 (EN)
- new net: J3.1 (Pin_1), U3.34 (RXD0)
- new net: J3.2 (Pin_2), U3.35 (TXD0)
- new net: R32.2, SW2.1
- new net: R32.1, SW1.2
- new net +3V3: J3.3 (Pin_3), R32.1, R32.2, U3.2 (3V3)
- new net IN1: U3.26 (IO4)
- new net IN2: U3.27 (IO16)
- new net IN3: U3.28 (IO17)
- new net IN4: U3.29 (IO5)
- new net IN5: U3.30 (IO18)
- new net IN6: U3.31 (IO19)
- no-connect marks 0 -> 17
Other:
- added sheet Fuente de alimentacion (Power.kicad_sch)
- added sheet Salidas_Potencia (Salidas_Potencia.kicad_sch)
